File: ElectricalLayoutV2.kicad_sch (KiCad schematic)
At the start: 47 parts, among them K1 3.3V-24V (40A), K2 Relay_SPST-NO, K3 Relay_SPST-NO, K4 Relay_SPST-NO, SW1 SW_Push, SW3 SW_Push, SW4 SW_Push, SW5 SW_Push, U1 DS18B20, U2 DS18B20, U3 DS18B20, U4 DS18B20, U5 DS18B20

Commit message: Start working on Electronics Box
Parts:
- added ARD1: ~, symbol Exocet_Electrical:Arduino
- added RELB1, RELB2, RELB3: ~, symbol Exocet_Electrical:Relay_Board
- added RPI1: ~, symbol Exocet_Electrical:Raspberry_Pi
Connections:
- net at DCC1. (-Vout): now also F6.1; no longer PROP1. (Vcc)
- net at MRG2.: now also FCC1. (Vcc); no longer FCC2. (Vcc)
- new net: FC3. (FC_SIG), FCC2. (Vcc) (x2)
- new net: DCC1. (-Vout), PROP1. (Vcc)
- new net: DCC1. (-Vout), MRG2., SW3.2
- new net: FCC1. (Vcc), FCC2. (Vcc), K1.14
- new net: FCC2. (Vcc), MRG2.
- new net: FC4. (FC_SIG), FCC1. (Vcc) (x2)
- new net: ARD1. (USB), RPI1. (USBv3_1)
- no-connect marks 4 -> 5

Commit message: First full version of 2024 electrical layout
Parts:
- removed BSB1: ~, symbol Exocet_Electrical:Busbar_4
- removed D4: D, symbol Device:D
- removed MRG1: 50A -> 100A, symbol Exocet_Electrical:Merger_2_1
- removed MRG2, MRG3: ~, symbol Exocet_Electrical:Merger_2_1
- added BSB1: 50A, symbol Exocet_Electrical:Busbar_3
- added BSB2: 50A, symbol Exocet_Electrical:Busbar_7
- added BSB3: 20A*, symbol Exocet_Electrical:Busbar_4
- added BSB4: 20A*, symbol Exocet_Electrical:Busbar_10
- added PCB1: ~, symbol Exocet_Electrical:PCB
- K1: value 3.3V-24V (40A) -> Coil: 24V, Contact: 40A
- R1: value 100Ω -> 500µΩ; Example (none) -> https://uk.rs-online.com/web/p/shunts/8103267; Name (none) -> Shunt Resistor; Note Max power: 6W -> (none)
- RELB1: Name (none) -> Actuators Relay Board
- RELB2: Name (none) -> Contactors Relay Board 1
- RELB3: Name (none) -> Contactors Relay Board 2
Connections:
- net AWG 12: now also BSB1.
- net AWG 8: now also BSB1.
- net at RELB3. (Vcc): now also BSB4.
- net at FCC2. (Vcc): now also D1.2 (A); no longer FC3. (FC_SIG)
- net at R1.1: now also BSB1.; no longer SW2.1
- net at R1.2: now also D3.1 (K)
- net at RELB1. (Vcc): now also BSB4.
- net at K2.14: now also D1.1 (K), D2.1 (K)
- net at K2.A1: now also RELB3. (Vcc)
- net at DCC1. (-Vout): now also F6.1; no longer PROP1. (Vcc)
- net at DCC1. (-Vout), SW3.2: now also FCC1. (Vcc), FCC2. (Vcc)
- net at F4.1, R3.2: now also K4.13, R2.2
- net at K3.A1: now also RELB2. (Vcc)
- net at K4.A1: now also RELB2. (Vcc)
- net at FCC1. (Vcc): now also FC4. (FC_SIG)
- net at RPI1. (USBv3_1): now also ARD1. (USB)
- net at ARD1. (USB): no longer RPI1. (USBv3_1)
- net at K1.A2: now also RELB3. (Vcc)
- net at F3.1: now also BSB4.
- net at RELB2. (Vcc): now also BSB4.
- removed net GND: B2.2 (-), CGND1. (GND), FCC1. (Vcc), FCC2. (Vcc), K1.A1, K2.A2, K3.A2, K4.A2
- new net: BSB4., RELB3. (Vcc)
- new net: FC3. (FC_SIG), FCC2. (Vcc) (x2)
- new net: BSB2., BSB3.
- new net: BSB3., PCB1. (SIG)
- new net: BSB4., RELB1. (Vcc)
- new net: BSB2., K2.A2
- new net: DCC1. (-Vout), PROP1. (Vcc)
- new net: BSB2., K3.A2
- new net: BSB2., FCC1. (Vcc), FCC2. (Vcc)
- new net: FCC1. (Vcc), FCC2. (Vcc), K1.14
- new net: BSB2., K4.A2
- new net: BSB2., K1.A1
- new net: B2.2 (-), BSB2., CGND1. (GND)
- new net: FC4. (FC_SIG), FCC1. (Vcc) (x2)
- new net: PCB1. (SIG), RPI1. (USBv3_1)
- new net: BSB4., PCB1. (SIG)
- new net: BSB4., RELB2. (Vcc)
- no-connect marks 5 -> 53
Other:
- note added: "AWG 21"
- note removed: "AWG ? (same as dead man's switch, max current = 250mA)"
- moved on the sheet: D1, F1, F2, F3, F4, R2, R3
