File: ElectricalLayoutV2.kicad_sch (KiCad schematic)
At the start: 21 parts, among them U1 DS18B20, U2 DS18B20, U3 DS18B20, U4 DS18B20

Commit message: essais
Connections:
- net at FCC1. (Vcc): no longer FC1. (FC_SIG)
- net at PROP1. (Vcc): now also DCC1. (-Vout), R4.2
- net at FCC2. (Vcc): now also FC2. (FC_SIG)
- new net: FC1. (FC_SIG), FCC1. (Vcc) (x2)
- new net: FC2. (FC_SIG), FCC2. (Vcc) (x2)
- now unconnected: FCC1. (Vcc)
Other:
- sheet Low Power Box ports: added TemperatureSensor_Battery, TemperatureSensor_H2Plate, TemperatureSensor_H2Tanks; removed TEMP_1, TEMP_2, TEMP_3
Changed lines of the file:
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@@
 	)
 	(symbol
-		(lib_name "Fuel_Cell_2")
+		(lib_name "Exocet_Electrical:Fuel_Cell")
 		(lib_id "Exocet_Electrical:Fuel_Cell")
 		(at 73.66 72.39 0)
@@
 	)
 	(symbol
+		(lib_name "Exocet_Electrical:Manometer")
 		(lib_id "Exocet_Electrical:Manometer")
 		(at 257.81 220.98 0)
@@
 	)
 	(symbol
+		(lib_name "Exocet_Electrical:Fuel_Cell_Controller")
 		(lib_id "Exocet_Electrical:Fuel_Cell_Controller")
 		(at 97.79 72.39 0)
@@
 			)
 		)
-		(property "Datasheet" "https://polymtlca0.sharepoint.com/:b:/s/Exocet/EXMM8dqsfHlBmM3m8eTcPocB8HjCPjjwPfi4r1bv40I5IQ?e=W05IQO"
+		(property "Datasheet" "~"
 			(at 35.814 77.47 90)
 			(effects
@@
 			)
 		)
-		(property "Description" ""
+		(property "Description" "Single-cell battery"
 			(at 34.29 77.47 0)
 			(effects
@@
 			)
 		)
-		(property "Datasheet" "https://polymtlca0.sharepoint.com/:b:/s/Exocet/EXMM8dqsfHlBmM3m8eTcPocB8HjCPjjwPfi4r1bv40I5IQ?e=W05IQO"
+		(property "Datasheet" "~"
 			(at 35.814 88.9 90)
 			(effects
@@
 			)
 		)
-		(property "Description" ""
+		(property "Description" "Single-cell battery"
 			(at 34.29 88.9 0)
 			(effects
@@
 	)
 	(symbol
+		(lib_name "Exocet_Electrical:Valve_Actuator")
 		(lib_id "Exocet_Electrical:Valve_Actuator")
 		(at 208.28 220.98 0)
@@
 	)
 	(symbol
-		(lib_name "Fuel_Cell_3")
 		(lib_id "Exocet_Electrical:Fuel_Cell")
 		(at 73.66 92.71 0)
@@
 		)
 		(fill
-			(color 0 0 0 0.0000)
+			(color 255 255 194 1.0000)
 		)
 		(property "Sheetname" "Low Power Box"
-			(at 212.344 16.002 0)
-			(effects
-				(font
-					(size 1.27 1.27)
-				)
-				(justify left bottom)
+			(at 212.09 15.24 0)
+			(effects
+				(font
+					(size 5 5)
+					(bold yes)
+				)
+				(justify left top)
 			)
 		)
@@
 			)
 		)
-		(pin "TEMP_3" bidirectional
+		(pin "TemperatureSensor_Battery" bidirectional
 			(at 334.01 111.76 0)
 			(effects
@@
 			)
 		)
-		(pin "TEMP_2" bidirectional
+		(pin "TemperatureSensor_H2Tanks" bidirectional
 			(at 334.01 91.44 0)
 			(effects
@@
 			)
 		)
-		(pin "TEMP_1" bidirectional
+		(pin "TemperatureSensor_H2Plate" bidirectional
 			(at 334.01 71.12 0)
 			(effects
@@
 		)
 		(fill
-			(color 0 0 0 0.0000)
+			(color 255 255 194 1.0000)
 		)
 		(property "Sheetname" "Dashboard"
-			(at 133.604 16.002 0)
-			(effects
-				(font
-					(size 1.27 1.27)
-				)
-				(justify left bottom)
+			(at 133.35 15.24 0)
+			(effects
+				(font
+					(size 5 5)
+					(bold yes)
+				)
+				(justify left top)
 			)
 		)
@@
 		)
 		(fill
-			(color 0 0 0 0.0000)
+			(color 255 255 194 1.0000)
 		)
 		(property "Sheetname" "High Power Box"
-			(at 14.224 131.572 0)
-			(effects
-				(font
-					(size 1.27 1.27)
+			(at 13.97 208.28 0)
+			(effects
+				(font
+					(size 5 5)
+					(bold yes)
 				)
 				(justify left bottom)
