File: dashboard.kicad_sch (KiCad schematic)
At the start: 7 parts, among them SW1 SW_Push, SW3 SW_Push, SW4 SW_Push

Commit message: Start low power box sheet
Changed lines of the file:
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@@
-		(color 0 0 0 0)
-	)
-	(junction
-		(at 110.49 95.25)
-		(diameter 0)
 		(color 0 0 0 0)
 	)
@@
 	(bus
 		(pts
-			(xy 86.36 95.25) (xy 110.49 95.25)
-		)
-		(stroke
-			(width 0)
-			(type default)
-		)
-	)
-	(bus
-		(pts
 			(xy 186.69 92.71) (xy 186.69 88.9)
 		)
@@
 		(pts
 			(xy 158.75 90.17) (xy 143.51 90.17)
-		)
-		(stroke
-			(width 0)
-			(type default)
-		)
-	)
-	(bus
-		(pts
-			(xy 86.36 95.25) (xy 86.36 118.11)
 		)
 		(stroke
@@
 			)
 		)
-	)
-	(hierarchical_label "THR_CTRL"
-		(shape passive)
-		(at 86.36 118.11 270)
-		(effects
-			(font
-				(size 1.27 1.27)
-			)
-			(justify right)
-		)
-		(property "Connector" "Gland"
-			(at 84.836 118.872 0)
-			(effects
-				(font
-					(size 1.27 1.27)
-				)
-				(justify right)
-			)
-		)

Commit message: Finalize layout
Parts:
- added ARD1: ~, symbol Exocet_Electrical:Arduino
Connections:
- net at ANT1. (SIG): now also ARD1. (USB)

Commit message: essais
Changed lines of the file:
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@@
+	)
+	(bus_entry
+		(at 86.36 74.93)
+		(size 2.54 2.54)
+		(stroke
+			(width 0)
+			(type default)
+		)
 	)
 	(bus_entry
@@
 	(bus_entry
 		(at 134.62 109.22)
+		(size 2.54 2.54)
+		(stroke
+			(width 0)
+			(type default)
+		)
+	)
+	(bus_entry
+		(at 86.36 72.39)
 		(size 2.54 2.54)
 		(stroke
@@
 	(wire
 		(pts
+			(xy 92.71 71.12) (xy 99.06 71.12)
+		)
+		(stroke
+			(width 0)
+			(type default)
+		)
+	)
+	(wire
+		(pts
 			(xy 162.56 109.22) (xy 162.56 113.03)
 		)
@@
 		)
 	)
+	(bus
+		(pts
+			(xy 88.9 77.47) (xy 88.9 80.01)
+		)
+		(stroke
+			(width 0)
+			(type default)
+		)
+	)
 	(wire
 		(pts
@@
 		)
 	)
+	(bus
+		(pts
+			(xy 88.9 74.93) (xy 88.9 77.47)
+		)
+		(stroke
+			(width 0)
+			(type default)
+		)
+	)
 	(wire
 		(pts
 			(xy 194.31 90.17) (xy 179.07 90.17)
+		)
+		(stroke
+			(width 0)
+			(type default)
+		)
+	)
+	(bus
+		(pts
+			(xy 99.06 71.12) (xy 99.06 74.93)
 		)
 		(stroke
@@
 			)
 		)
-		(property "Description" ""
+		(property "Description" "Push button switch, generic, two pins"
 			(at 170.18 109.22 0)
 			(effects
