File: high_power_box.kicad_sch (KiCad schematic)
At the start: 25 parts, among them K1 SPST-NO, 24V, 50A, K2 DCNLEV100, K3 DCNLEV100, K4 SPST-NO, 24V, 30A, K5 DCNLEV100, K6 SPST-NO, 24V, 30A, SW5 SW_Push

Commit message: essais
Parts:
- K4, K6: footprint (none) -> Relay_THT:Relay_SPST_RAYEX-L90AS
Connections:
- net at C3.: no longer C7.
- net at C1.: now also K1.13
- net at BSEN1. (~{ALCC}): now also F2.1; no longer C1.
- new net: C3., C7.
- new net: BSEN1. (~{ALCC}), C1.
Changed lines of the file:
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@@
 			)
 		)
-		(property "Datasheet" ""
+		(property "Datasheet" "~"
 			(at 170.18 140.97 0)
 			(effects
@@
 			)
 		)
-		(property "Description" ""
+		(property "Description" "Relay SPST, Normally Open, EN50005"
 			(at 170.18 140.97 0)
 			(effects
@@
 			)
 		)
-		(property "Datasheet" ""
+		(property "Datasheet" "~"
 			(at 190.5 143.51 0)
 			(effects
@@
 			)
 		)
-		(property "Description" ""
+		(property "Description" "Resistor"
 			(at 190.5 143.51 0)
 			(effects
@@
 			)
 		)
-		(property "Datasheet" ""
+		(property "Datasheet" "~"
 			(at 133.35 140.97 0)
 			(effects
@@
 			)
 		)
-		(property "Description" ""
+		(property "Description" "Relay SPST, Normally Open, EN50005"
 			(at 133.35 140.97 0)
 			(effects
@@
 			)
 		)
-		(property "Datasheet" ""
+		(property "Datasheet" "~"
 			(at 104.14 140.97 0)
 			(effects
@@
 			)
 		)
-		(property "Description" ""
+		(property "Description" "Relay SPST, Normally Open, EN50005"
 			(at 104.14 140.97 0)
 			(effects
@@
 			)
 		)
-		(property "Datasheet" ""
+		(property "Datasheet" "~"
 			(at 172.72 121.92 0)
 			(effects
@@
 			)
 		)
-		(property "Description" ""
+		(property "Description" "Resistor"
 			(at 172.72 121.92 0)
 			(effects
@@
 			)
 		)
-		(property "Footprint" ""
+		(property "Footprint" "Relay_THT:Relay_SPST_RAYEX-L90AS"
 			(at 144.78 50.8 0)
 			(effects
@@
 			)
 		)
-		(property "Datasheet" ""
+		(property "Datasheet" "https://a3.sofastcdn.com/attachment/7jioKBjnRiiSrjrjknRiwS77gwbf3zmp/L90-SERIES.pdf"
 			(at 142.24 44.45 0)
 			(effects
@@
 			)
 		)
-		(property "Description" ""
+		(property "Description" "Power relay, Without Common Terminal between coil terminals, NO, SPST, 30A"
 			(at 146.05 62.23 0)
 			(effects
@@
 			)
 		)
-		(property "Footprint" ""
+		(property "Footprint" "Relay_THT:Relay_SPST_RAYEX-L90AS"
 			(at 180.34 50.8 0)
 			(effects
@@
 			)
 		)
-		(property "Datasheet" ""
+		(property "Datasheet" "https://a3.sofastcdn.com/attachment/7jioKBjnRiiSrjrjknRiwS77gwbf3zmp/L90-SERIES.pdf"
 			(at 177.8 44.45 0)
 			(effects
@@
 			)
 		)
-		(property "Description" ""
+		(property "Description" "Power relay, Without Common Terminal between coil terminals, NO, SPST, 30A"
 			(at 181.61 62.23 0)
 			(effects
@@
 			)
 		)
-		(property "Datasheet" ""
+		(property "Datasheet" "~"
 			(at 74.93 52.07 0)
 			(effects
@@
 			)
 		)
-		(property "Description" ""
+		(property "Description" "Relay SPST, Normally Open, EN50005"
 			(at 74.93 52.07 0)
 			(effects
@@
 			)
 		)
-		(property "Description" ""
+		(property "Description" "Fuse"
 			(at 39.37 46.99 0)
 			(effects
