File: low_power_box.kicad_sch (KiCad schematic)
At the start: 8 parts

Commit message: Complete Low Power Box
Parts:
- removed BSB1: 20A, symbol Exocet_Electrical:Busbar_4
- removed BSB2: 20A, symbol Exocet_Electrical:Busbar_10
- added BSEN1: ~, symbol Exocet_Electrical:Battery_Sense
- added DC5V1: ~, symbol Exocet_Electrical:DC-DC_24V_5V
- added RELB4: ~, symbol Exocet_Electrical:Relay_Board
Connections:
- net +24V: now reaches RELB1. (Vcc)
- net +24V: now also RELB2. (Vcc), RELB3. (Vcc), DC5V1. (-Vout), RELB4. (Vcc)
- net at RPI1. (USBv3_1): now also ARD1. (USB); no longer PCB1. (SIG)
- net at ARD1. (USB): no longer RPI1. (USBv3_1)
- new net: BSEN1. (~{ALCC}), PCB1. (~{ALCC}) (x5)
- new net: DC5V1. (-Vout), PCB1. (~{ALCC}) (x2)
- new net: PCB1. (~{ALCC}), RPI1. (USBv3_1)
- new net GND: DC5V1. (-Vout)
- now unconnected: PCB1. (SIG)
- no-connect marks 33 -> 21
Other:
- note added: "Busbar"
- note removed: "Electronics Box"

Commit message: Finalize layout
Parts:
- removed ARD1: ~, symbol Exocet_Electrical:Arduino
- removed BSEN1: ~, symbol Exocet_Electrical:Battery_Sense
Connections:
- net at RPI1. (USBv3_1): now also PCB1. (~{ALCC})
- new net: DC5V1. (-Vout), PCB1. (~{ALCC}) (x2)
- now unconnected: PCB1. (~{ALCC}), PCB1. (~{ALCC}), PCB1. (~{ALCC}), PCB1. (~{ALCC}), PCB1. (~{ALCC}), PCB1. (~{ALCC}), PCB1. (~{ALCC})
- no-connect marks 21 -> 22
Other:
- title: (none) -> Low Power Box Layout

Commit message: essais
Parts:
- added C10: JST PH, symbol Exocet_Electrical:Connector_2pins
- added C8: 3 pins, symbol Exocet_Electrical:Connector_3pins
- added C9: JST PH, symbol Exocet_Electrical:Connector_5pins
- added U5: ~, symbol Exocet_Electrical:PCB2
Connections:
- net at PCB1. (~{ALCC}): no longer DC5V1. (-Vout)
- net at RPI1. (USBv3_1): now also PCB1. (~{ALCC})
- new net: C9.1, U5. (~{ALCC})
- new net: C9.2, U5. (~{ALCC})
- new net: C9.3, U5. (~{ALCC})
- new net: C9.4, U5. (~{ALCC})
- new net: C9.5, U5. (~{ALCC})
- new net: C8.1, U5. (~{ALCC})
- new net: C8.2, U5. (~{ALCC})
- new net: C8.3, U5. (~{ALCC})
- new net: C10.1, U5. (~{ALCC})
- new net: C10.2, U5. (~{ALCC})
- new net: DC5V1. (-Vout), PCB1. (~{ALCC}) (x2)
- now unconnected: PCB1. (~{ALCC}), PCB1. (~{ALCC})
Other:
- note added: "Low Power Box"
- moved on the sheet: DC5V1
